Commit message: [Feat] Continue to add ur10e configs to test it.

File: src/ur10e_anima/ur10e_description/urdf/inc/ur_macro.xacro (robot description, xacro)
@@ -297,5 +297,5 @@
            the UR controller.
       -->
-      <origin xyz="0 0 0" rpy="0 0 ${pi}"/>
+      <origin xyz="0 0 0" rpy="0 0 ${pi/2.0}"/>
       <parent link="${prefix}base_link"/>
       <child link="${prefix}base"/>

Commit message: [Fix] Solve rotation issue on the ur10e urdf.

File: src/ur10e_anima/ur10e_description/urdf/inc/ur_macro.xacro (robot description, xacro)
@@ -215,5 +215,5 @@
            link/frame) to introduce the necessary rotation over Z (of pi rad).
       -->
-      <origin xyz="0 0 0" rpy="0 0 ${pi}" />
+      <origin xyz="0 0 0" rpy="0 0 ${pi/2.0}" />
     </joint>
     <joint name="${prefix}shoulder_pan_joint" type="revolute">
