Commit message: [Feat] Add end effector sensor and end effector tools as parameters. The sensor is hardcoded for each UR since our hardware has clear sensor definition.

File: src/ur-package/ur_description/urdf/inc/ur10e_macro.xacro (robot description, xacro)
@@ -26,5 +26,7 @@
    safety_limits:=false
    safety_pos_margin:=0.15
-   safety_k_position:=20"
+   safety_k_position:=20
+   ee_force_torque:=none
+   ee_tool:=none"
   >
     <xacro:include filename="$(find ur_description)/urdf/inc/ur_macro.xacro"/>
@@ -39,4 +41,6 @@
       safety_pos_margin="${safety_pos_margin}"
       safety_k_position="${safety_k_position}"
+      ee_force_torque="${ee_force_torque}"
+      ee_tool="${ee_tool}"
     />
   </xacro:macro>

File: src/ur-package/ur_description/urdf/inc/ur5_macro.xacro (robot description, xacro)
@@ -17,6 +17,5 @@
           real robot.
   -->
-  <xacro:macro name="ur5_robot"
-    params="
+  <xacro:macro name="ur5_robot" params="
    prefix
    joint_limits_parameters_file:='$(find ur_description)/config/ur5/joint_limits.yaml'
@@ -28,4 +27,5 @@
    safety_pos_margin:=0.15
    safety_k_position:=20
+   ee_force_torque:=true
    ee_tool:=none"
   >
@@ -41,4 +41,5 @@
       safety_pos_margin="${safety_pos_margin}"
       safety_k_position="${safety_k_position}"
+      ee_force_torque="${ee_force_torque}"
       ee_tool="${ee_tool}"
     />

File: src/ur-package/ur_description/urdf/inc/ur_macro.xacro (robot description, xacro)
@@ -55,5 +55,6 @@
     safety_pos_margin:=0.15
     safety_k_position:=20
-    ee_tool:=none"
+    ee_tool:=none
+    ee_force_torque:=none"
   >
     <!-- Load configuration data from the provided .yaml files -->
@@ -344,39 +345,11 @@
       <child link="${prefix}tool0" />
     </joint>
-    <!-- ROS-Industrial 'sensor' frame: attachment point for force-torque sensors -->
-    <!-- TODO Add the force torque sensor using a parameter -->
-    <link name="${prefix}sensor">
-      <visual>
-        <geometry>
-          <mesh
-            filename="package://ur_description/meshes/ur5/visual/force_torque.stl"
-            scale="1 1 1" />
-        </geometry>
-        <!-- Small offset to avoid any collisions between adjacent -->
-        <origin rpy="0 0 0" xyz="0 0 0" />
-        <material name="LightGrey" />
-      </visual>
-      <inertial>
-        <mass value="0.5" />
-        <inertia ixx="0.1" ixy="-0.000000" ixz="-0.000000" iyy="0.1" iyz="-0.000000"
-          izz="0.1" />
-        <origin rpy="0 0 0" xyz="0.0 0.0 0.0" />
-      </inertial>
-      <collision>
-        <geometry>
-          <mesh
-            filename="package://ur_description/meshes/ur5/collision/force_torque.stl"
-            scale="1 1 1" />
-        </geometry>
-        <!-- Small z offset to avoid any collisions between adjacent -->
-        <origin rpy="0 0 0" xyz="0 0 0" />
-      </collision>
-    </link>
-    <joint name="${prefix}tool0-sensor" type="fixed">
-      <!-- default toolframe: X+ left, Y+ up, Z+ front -->
-      <origin xyz="0 0 0.035" rpy="0 0 0" />
-      <parent link="${prefix}tool0" />
-      <child link="${prefix}sensor" />
-    </joint>
+    <!-- Add force torque sensor -->
+    <xacro:property name="sensor_frame" value="tool0" />
+    <xacro:if value="${ee_force_torque != 'none'}">
+      <xacro:property name="sensor_frame" value="sensor" />
+      <xacro:include filename="$(find ur_description)/urdf/force_torque.urdf.xacro" />
+    </xacro:if>
+    <!-- Add end-effector tool -->
     <xacro:if value="${ee_tool != 'none'}">
       <xacro:include filename="$(find ur_description)/urdf/tools.urdf.xacro" />
@@ -384,6 +357,6 @@
     <xacro:if value="${ee_tool == 'none'}">
       <link name="${prefix}virtual_link" />
-      <joint name="${prefix}sensor-virtual_link" type="fixed">
-        <parent link="${prefix}sensor" />
+      <joint name="${prefix}${sensor_frame}-virtual_link" type="fixed">
+        <parent link="${prefix}${sensor_frame}" />
         <child link="${prefix}virtual_link" />
         <origin rpy="0 0 0" xyz="0 0 0" />

File: src/ur-package/ur_description/urdf/tools.urdf.xacro (robot description, xacro)
@@ -3,5 +3,5 @@
     <xacro:include filename="$(find experiments)/urdf/ee_logi_laser.urdf.xacro" />
     <xacro:if value="${ee_tool == 'logi_laser'}">
-        <xacro:ee_laser prefix="${prefix}" />
+        <xacro:ee_laser prefix="${prefix}" sensor_frame="${sensor_frame}" />
     </xacro:if>
 </robot>

File: src/ur-package/ur_description/urdf/ur.xacro (robot description, xacro)
@@ -13,13 +13,14 @@
          - hardware_interface/EffortJointInterface
    -->
-      <xacro:arg name="transmission_hw_interface"
-            default="hardware_interface/PositionJointInterface" />
+      <xacro:arg name="transmission_hw_interface" default="hardware_interface/PositionJointInterface" />
       <xacro:arg name="safety_limits" default="false" />
       <xacro:arg name="safety_pos_margin" default="0.15" />
       <xacro:arg name="safety_k_position" default="20" />
+      <xacro:arg name="ee_force_torque" default="none" />
       <xacro:arg name="ee_tool" default="none" />
       <!-- arm -->
       <xacro:ur_robot
             prefix=""
+            ee_force_torque="$(arg ee_force_torque)"
             ee_tool="$(arg ee_tool)"
             joint_limits_parameters_file="$(arg joint_limit_params)"

File: src/ur-package/ur_description/urdf/ur10e.xacro (robot description, xacro)
@@ -1,4 +1,6 @@
 <?xml version="1.0"?>
 <robot xmlns:xacro="http://wiki.ros.org/xacro" name="ur10e_robot">
+  <xacro:arg name="ee_force_torque" default="none" />
+  <xacro:arg name="ee_tool" default="none" />
   <!--
     This is a convenience top-level xacro which loads the macro for the UR10e
@@ -15,4 +17,4 @@
   -->
   <xacro:include filename="$(find ur_description)/urdf/inc/ur10e_macro.xacro"/>
-  <xacro:ur10e_robot prefix="" />
+  <xacro:ur10e_robot prefix="" ee_tool="$(arg ee_tool)" ee_force_torque="$(arg ee_force_torque)" />
 </robot>

File: src/ur-package/ur_description/urdf/ur5.xacro (robot description, xacro)
@@ -1,4 +1,5 @@
 <?xml version="1.0"?>
 <robot xmlns:xacro="http://wiki.ros.org/xacro" name="ur5_robot">
+  <xacro:arg name="ee_force_torque" default="true" />
   <xacro:arg name="ee_tool" default="none" />
   <!--
@@ -16,4 +17,4 @@
   -->
   <xacro:include filename="$(find ur_description)/urdf/inc/ur5_macro.xacro" />
-  <xacro:ur5_robot prefix="" ee_tool="$(arg ee_tool)" />
+  <xacro:ur5_robot prefix="" ee_tool="$(arg ee_tool)" ee_force_torque="$(arg ee_force_torque)" />
 </robot>
